File: pq_obc&comms/PQ_OBC&COMMS/PQ_OBC&COMMS.kicad_sch (KiCad schematic)
At the start: 66 parts, among them J1 Conn_01x10, J2 Conn_01x10, J3 Conn_01x10, J4 Conn_01x10, J6 U.FL-R-SMT-1_10_, U1 STM32L162RETx, U2 SX1262IMLTRT, U3 BD2232G-GTR, U4 BD2232G-GTR, U5 RFswitch, U7 BD2232G-GTR, X1 12MHz, X2 FA-128_32.0000MF20X-K5, X3 32.768KHz

Commit message: change organization
Other:
- moved on the sheet: C12, L6
Changed lines of the file:
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@@
   (junction (at 241.3 74.93) (diameter 0) (color 0 0 0 0)
   )
-  (junction (at 151.13 212.09) (diameter 0) (color 0 0 0 0)
+  (junction (at 151.13 205.74) (diameter 0) (color 0 0 0 0)
   )
   (junction (at 355.6 162.56) (diameter 0) (color 0 0 0 0)
@@
     (stroke (width 0) (type default) (color 0 0 0 0))
   )
-  (wire (pts (xy 146.05 212.09) (xy 151.13 212.09))
+  (wire (pts (xy 146.05 205.74) (xy 151.13 205.74))
     (stroke (width 0) (type default) (color 0 0 0 0))
   )
@@
     (stroke (width 0) (type default) (color 0 0 0 0))
   )
-  (polyline (pts (xy 193.04 144.78) (xy 193.04 13.97))
+  (polyline (pts (xy 193.04 144.78) (xy 193.04 20.32))
     (stroke (width 0.254) (type solid) (color 0 0 0 0))
   )
@@
     (stroke (width 0) (type default) (color 0 0 0 0))
   )
-  (polyline (pts (xy 193.04 13.97) (xy 193.04 144.78))
+  (polyline (pts (xy 193.04 20.32) (xy 193.04 144.78))
     (stroke (width 0.254) (type solid) (color 0 0 0 0))
   )
@@
     (stroke (width 0) (type default) (color 0 0 0 0))
   )
-  (polyline (pts (xy 369.57 13.97) (xy 369.57 144.78))
+  (polyline (pts (xy 369.57 20.32) (xy 369.57 144.78))
     (stroke (width 0.254) (type solid) (color 0 0 0 0))
   )
@@
     (stroke (width 0) (type default) (color 0 0 0 0))
   )
-  (polyline (pts (xy 369.57 13.97) (xy 293.37 13.97))
+  (polyline (pts (xy 369.57 20.32) (xy 293.37 20.32))
     (stroke (width 0.254) (type solid) (color 0 0 0 0))
   )
@@
     (stroke (width 0) (type default) (color 0 0 0 0))
   )
-  (polyline (pts (xy 293.37 144.78) (xy 293.37 13.97))
+  (polyline (pts (xy 293.37 144.78) (xy 293.37 20.32))
     (stroke (width 0.254) (type solid) (color 0 0 0 0))
   )
@@
     (stroke (width 0.254) (type default) (color 0 0 0 0))
   )
-  (polyline (pts (xy 293.37 13.97) (xy 293.37 144.78))
+  (polyline (pts (xy 293.37 20.32) (xy 293.37 144.78))
     (stroke (width 0.254) (type solid) (color 0 0 0 0))
   )
@@
     (stroke (width 0) (type default) (color 0 0 0 0))
   )
-  (polyline (pts (xy 193.04 13.97) (xy 36.83 13.97))
+  (polyline (pts (xy 193.04 20.32) (xy 36.83 20.32))
     (stroke (width 0.254) (type solid) (color 0 0 0 0))
   )
@@
     (stroke (width 0) (type default) (color 0 0 0 0))
   )
-  (polyline (pts (xy 36.83 144.78) (xy 36.83 13.97))
+  (polyline (pts (xy 36.83 144.78) (xy 36.83 20.32))
     (stroke (width 0.254) (type solid) (color 0 0 0 0))
   )
@@
     (stroke (width 0) (type default) (color 0 0 0 0))
   )
-  (polyline (pts (xy 293.37 13.97) (xy 193.04 13.97))
+  (polyline (pts (xy 293.37 20.32) (xy 193.04 20.32))
     (stroke (width 0.254) (type solid) (color 0 0 0 0))
   )
@@
     (stroke (width 0) (type default) (color 0 0 0 0))
   )
-  (wire (pts (xy 151.13 198.12) (xy 151.13 204.47))
-    (stroke (width 0) (type default) (color 0 0 0 0))
-  )
   (wire (pts (xy 356.87 105.41) (xy 354.33 105.41))
     (stroke (width 0.254) (type default) (color 0 0 0 0))
@@
     (stroke (width 0) (type default) (color 0 0 0 0))
   )
-  (wire (pts (xy 146.05 180.34) (xy 146.05 212.09))
+  (wire (pts (xy 146.05 180.34) (xy 146.05 205.74))
     (stroke (width 0) (type default) (color 0 0 0 0))
   )
@@
     (pin "")
   )
-  (symbol (lib_id "Device:C") (at 151.13 215.9 0) (unit 1)
-    (in_bom yes) (on_board yes) (fields_autoplaced)
-    (property "Reference" "C12" (id 0) (at 154.94 214.8211 0)
+  (symbol (lib_id "Device:C") (at 151.13 209.55 0) (unit 1)
+    (in_bom yes) (on_board yes)
+    (property "Reference" "C12" (id 0) (at 154.94 208.4711 0)
       (effects (font (size 1.27 1.27)) (justify left))
     )
-    (property "Value" "1.8pF" (id 1) (at 154.94 217.3611 0)
+    (property "Value" "1.8pF" (id 1) (at 154.94 211.0111 0)
       (effects (font (size 1.27 1.27)) (justify left))
     )
-    (property "Footprint" "" (id 2) (at 152.0952 219.71 0)
+    (property "Footprint" "" (id 2) (at 152.0952 213.36 0)
       (effects (font (size 1.27 1.27)) hide)
     )
-    (property "Datasheet" "~" (id 3) (at 151.13 215.9 0)
+    (property "Datasheet" "~" (id 3) (at 151.13 209.55 0)
       (effects (font (size 1.27 1.27)) hide)
     )
-    (property "CONTRIBUTOR" "danielCOMMS" (id 4) (at 151.13 215.9 0)
+    (property "CONTRIBUTOR" "danielCOMMS" (id 4) (at 151.13 209.55 0)
       (effects (font (size 1.27 1.27)) (justify left bottom) hide)
     )
-    (property "SPICEPRE" "C" (id 5) (at 151.13 215.9 0)
+    (property "SPICEPRE" "C" (id 5) (at 151.13 209.55 0)
       (effects (font (size 1.27 1.27)) (justify left bottom) hide)
     )
-    (property "SPICESYMBOLNAME" "GRM1555C1H1R8BA01D" (id 6) (at 151.13 215.9 0)
+    (property "SPICESYMBOLNAME" "GRM1555C1H1R8BA01D" (id 6) (at 151.13 209.55 0)
       (effects (font (size 1.27 1.27)) (justify left bottom) hide)
     )
-    (property "BOM_MANUFACTURER PART" "" (id 7) (at 151.13 215.9 0)
+    (property "BOM_MANUFACTURER PART" "" (id 7) (at 151.13 209.55 0)
       (effects (font (size 1.27 1.27)) (justify left bottom) hide)
     )
@@
     (pin "2")
   )
-  (symbol (lib_id "Device:L") (at 151.13 208.28 0) (unit 1)
+  (symbol (lib_id "Device:L") (at 151.13 201.93 0) (unit 1)
     (in_bom yes) (on_board yes) (fields_autoplaced)
-    (property "Reference" "L6" (id 0) (at 152.4 207.0099 0)
+    (property "Reference" "L6" (id 0) (at 152.4 200.6599 0)
       (effects (font (size 1.27 1.27)) (justify left))
     )
-    (property "Value" "15nH" (id 1) (at 152.4 209.5499 0)
+    (property "Value" "15nH" (id 1) (at 152.4 203.1999 0)
       (effects (font (size 1.27 1.27)) (justify left))
     )
-    (property "Footprint" "" (id 2) (at 151.13 208.28 0)
+    (property "Footprint" "" (id 2) (at 151.13 201.93 0)
       (effects (font (size 1.27 1.27)) hide)
     )
-    (property "Datasheet" "~" (id 3) (at 151.13 208.28 0)
+    (property "Datasheet" "~" (id 3) (at 151.13 201.93 0)
       (effects (font (size 1.27 1.27)) hide)
     )
-    (property "CONTRIBUTOR" "danielCOMMS" (id 4) (at 151.13 208.28 0)
+    (property "CONTRIBUTOR" "danielCOMMS" (id 4) (at 151.13 201.93 0)
       (effects (font (size 1.27 1.27)) (justify left bottom) hide)
     )
-    (property "SPICEPRE" "L" (id 5) (at 151.13 208.28 0)
+    (property "SPICEPRE" "L" (id 5) (at 151.13 201.93 0)
       (effects (font (size 1.27 1.27)) (justify left bottom) hide)
     )
-    (property "SPICESYMBOLNAME" "LQW15AN15NH00D" (id 6) (at 151.13 208.28 0)
+    (property "SPICESYMBOLNAME" "LQW15AN15NH00D" (id 6) (at 151.13 201.93 0)
       (effects (font (size 1.27 1.27)) (justify left bottom) hide)
     )
-    (property "BOM_MANUFACTURER PART" "" (id 7) (at 151.13 208.28 0)
+    (property "BOM_MANUFACTURER PART" "" (id 7) (at 151.13 201.93 0)
       (effects (font (size 1.27 1.27)) (justify left bottom) hide)
     )
@@
     (pin "1")
   )
-  (symbol (lib_id "COMMS-altium-import:GND") (at 151.13 219.71 0) (unit 1)
-    (in_bom yes) (on_board yes) (fields_autoplaced)
-    (property "Reference" "#PWR0107" (id 0) (at 151.13 219.71 0)
+  (symbol (lib_id "COMMS-altium-import:GND") (at 151.13 213.36 0) (unit 1)
+    (in_bom yes) (on_board yes)
+    (property "Reference" "#PWR0107" (id 0) (at 151.13 213.36 0)
       (effects (font (size 1.27 1.27)) hide)
     )
-    (property "Value" "GND" (id 1) (at 151.13 227.33 0))
-    (property "Footprint" "" (id 2) (at 151.13 219.71 0)
+    (property "Value" "GND" (id 1) (at 151.13 220.98 0))
+    (property "Footprint" "" (id 2) (at 151.13 213.36 0)
       (effects (font (size 1.27 1.27)) hide)
     )
-    (property "Datasheet" "" (id 3) (at 151.13 219.71 0)
+    (property "Datasheet" "" (id 3) (at 151.13 213.36 0)
       (effects (font (size 1.27 1.27)) hide)
     )
