File: pq_obc&comms/PQ_OBC&COMMSv3/PQ_OBC&COMMSv3.kicad_pcb (KiCad board)
At the start: 4 copper layers, 40 x 40 mm, 66 parts, among them J1 Conn_01x10, J2 Conn_01x10, J3 Conn_01x10, J4 Conn_01x10, J6 U.FL-R-SMT-1_10_, U1 STM32L162RETx, U2 SX1262IMLTRT, U3 BD2232G-GTR, U4 BD2232G-GTR, U5 RFswitch, U7 BD2232G-GTR, X1 12MHz, X2 FA-128_32.0000MF20X-K5, X3 32.768KHz

Commit message: hw revision of OBC
Parts:
- removed C44: 1uF, easyeda:CAPC1608X90N
- removed U4: BD2232G-GTR, easyeda:SSOP-5_L3.0-W1.6-P0.95-LS2.8-TL
- C1, C10, C11, C12, C2, C4, C5, C6, C7, C8, C9: footprint easyeda:CAPC1005X55N -> Capacitor_SMD:C_0402_1005Metric
- C14, C15, C16, C17, C18: footprint easyeda:CAPC1608X90N -> Capacitor_SMD:C_0603_1608Metric
- C27, C28, C31, C32, C33, C34, C35, C36, C37, C40, C41, C42, C43, C45: footprint easyeda:CAPC1608X90N -> Capacitor_SMD:C_0603_1608Metric; moved to B.Cu
- J6: value U.FL-R-SMT-1_10_ -> U.FL-R-SMT-1_10; footprint easyeda:U.FL-R-SMT-1(10) -> Connector_Coaxial:U.FL_Hirose_U.FL-R-SMT-1_Vertical
- L1, L3, L4, L5, L6: footprint easyeda:LQW15CNR20J00B -> Inductor_SMD:L_0402_1005Metric
- L2: footprint Resistor_SMD:R_0402_1005Metric -> Inductor_SMD:L_0402_1005Metric
- L7: footprint easyeda:INDC2012X145N -> Inductor_SMD:L_0805_2012Metric
- R3, R4: footprint easyeda:RESC1608X55N -> Resistor_SMD:R_0603_1608Metric
- R6, R7, R8: footprint easyeda:RESC1608X55N -> Resistor_SMD:R_0603_1608Metric; moved to B.Cu
- TP1: renamed from PROBE1; value MS-156C -> CoaxialSwitch_Testpoint
- U1: value STM32L162RETx -> STM32L476RGTx; footprint easyeda:STM-LQFP64 -> Package_QFP:LQFP-64_10x10mm_P0.5mm
- U2: footprint easyeda:QFN-24_L4.0-W4.0-P0.50-BL-EP2.6 -> Package_DFN_QFN:QFN-24-1EP_4x4mm_P0.5mm_EP2.6x2.6mm
- U3, U7: footprint easyeda:SSOP-5_L3.0-W1.6-P0.95-LS2.8-TL -> Package_SO:TSOP-5_1.65x3.05mm_P0.95mm; moved to B.Cu
- moved J4 22.9 mm to (110.6, 79.8), turned to -90 degrees
- moved J2 22.9 mm to (82.6, 74.7), turned to 180 degrees
- moved L6 1.09 mm to (105.9, 59.3)
- moved L3 1.03 mm to (108.3, 64.1)
- moved L4 1.03 mm to (108.3, 68.9)
- moved L5 0.94 mm to (104.5, 72.8)
- moved L1 0.91 mm to (108.8, 62.6)
- turned C27 to 0 degrees
- turned C31 to 180 degrees
- turned C32 to 180 degrees
- turned C33 to 180 degrees
- turned C34 to 180 degrees
- turned C35 to 180 degrees
- turned C36 to 180 degrees
- turned C37 to 180 degrees
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Connections:
- net BURNCOMMS_OBC renamed /PoL_BURN_EN
- net DIO1 renamed /DIO1
- net MISO renamed /MISO
- net MOSI renamed /MOSI
- net NRESET renamed /SX1262_NRST
- net NSS renamed /SX1262_NSS
- net Net-(R6-Pad1) renamed /Boot0
- net PALE renamed STM32_PB3
- net PDATA renamed STM32_PD2
- net P/L2BURN_OBC renamed STM32_PA15
- net P/L_POWER_OBC renamed /PoL_P/L_EN
- net RX renamed UART_RX
- net SCK renamed /SCK
- net TX renamed UART_TX
- C10 pad 1: Net-(C10-Pad1) -> Net-(J6-Pad1)
- C14 pad 1: Net-(C14-Pad1) -> Net-(U5-Pad4)
- C43 pad 1: GND -> VCC
- C43 pad 2: VCC -> GND
- D1 pad 2: Net-(D1-Pad2) -> VCC_UMBILICAL
- J1 pad 10: Net-(D1-Pad2) -> VCC
- J1 pad 4: unconnected-(J1-Pad4) -> KILLSWITCH+
- J1 pad 6: unconnected-(J1-Pad6) -> BATT-
- J2 pad 1: PCLK -> SOLAR_X
- J2 pad 10: SOLAR_X -> STM32_PA2
- J2 pad 2: ADC_PL2 -> unconnected-(J2-Pad2)
- J2 pad 3: DAC_PL2 -> CLPROG
- J2 pad 4: SWCLK -> CHRGOFF
- J2 pad 5: SWDIO -> NRST
- J2 pad 6: NRST -> SWDIO
- J2 pad 7: CHGOFF -> SWCLK
- J2 pad 8: CLPROG -> DAC_PL
- J2 pad 9: MPPT_X -> ADC_PL
- J3 pad 10: RST -> unconnected-(J3-Pad10)
- J3 pad 7: SEL -> HEATER_EN
- J3 pad 8: HEATER -> HEATER_PWR
- J4 pad 1: CHRG -> SOLAR_Z
- J4 pad 10: SOLAR_Z -> CHRG
- J4 pad 2: FAULT -> unconnected-(J4-Pad2)
- J4 pad 3: VCC_TEST1 -> unconnected-(J4-Pad3)
- J4 pad 4: SEL_PH3 -> RST_DRIVERS
- J4 pad 5: P/L_POWER -> ADC_PH
- J4 pad 6: ADC_PH1 -> P/L_POWER
- J4 pad 7: RST_DRIVERS -> SEL_PH0
- J4 pad 8: MPPT_Y -> VCC_UMBILICAL
- J4 pad 9: MPPT_Z -> FAULT
- J6 pad 1: GND -> Net-(J6-Pad1)
- L5 pad 2: Net-(C10-Pad1) -> Net-(J6-Pad1)
- R4 pad 2: Net-(C14-Pad1) -> Net-(U5-Pad4)
- U1 pad 15: ADC_PL2 -> ADC_PL
- U1 pad 16: PCLK -> STM32_PA2
- U1 pad 17: SEL -> unconnected-(U1-Pad17)
- U1 pad 21: DAC_PL2 -> DAC_PL
- U1 pad 23: CHRG -> MPPT_Z
- U1 pad 25: ADC_PH1 -> ADC_PH
- U1 pad 26: RST -> EPS_RST
- U1 pad 28: MPPT_Z -> CHRG
- U1 pad 29: HEATER -> HEATER_EN
- U1 pad 41: BUSY -> /BUSY
- U1 pad 5: OSC_OUT -> OSC_IN
- U1 pad 6: OSC_IN -> OSC_OUT
- U2 pad 14: BUSY -> /SX1262_BUSY
Routing:
- net HEATER_EN: track 0.00 -> 56.5 mm, vias 0 -> 3
- net RST: track 37.1 -> 0.00 mm
- net SEL: track 33.5 -> 0.00 mm, vias 2 -> 0
- net /PoL_P/L_EN: track 34.2 -> 4.72 mm
- net P/L_POWER: track 2.84 -> 32.3 mm
- net HEATER: track 23.0 -> 0.00 mm, vias 1 -> 0
- net unconnected-(J4-Pad3): track 0.00 -> 21.8 mm
- net MPPT_Y: track 21.8 -> 0.00 mm
- net DAC_PL2: track 19.2 -> 0.00 mm, vias 1 -> 0
- net DAC_PL: track 0.00 -> 19.2 mm, vias 0 -> 1
- net ADC_PH1: track 18.8 -> 0.00 mm
- net ADC_PH: track 0.00 -> 18.8 mm
- net STM32_PA2: track 0.00 -> 16.0 mm
- net PCLK: track 16.0 -> 0.00 mm
- net unconnected-(J2-Pad2): track 0.00 -> 14.0 mm
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Other:
- board text added: "+X"
- board text added: "+Z"
- board text added: "-X"
- board text added: "-Z"
- board text removed: "12MHz"
- board text removed: "32.7KHz"
- board text removed: "32MHz"
- board text removed: "BD2232G"
- board text removed: "BurnCOMMS"
- board text removed: "D-VCCTest"
- board text removed: "OBC-COMMS"
- board text removed: "PL2BURN"
- board text removed: "PL2VCC"
- board text removed: "STM32L162RE"
- board text removed: "SX1262"
