File: pq_obc&comms/PQ_OBC&COMMSv3/PQ_OBC&COMMSv3.kicad_sch (KiCad schematic)
At the start: 66 parts, among them J1 Conn_01x10, J2 Conn_01x10, J3 Conn_01x10, J4 Conn_01x10, J6 U.FL-R-SMT-1_10_, U1 STM32L162RETx, U2 SX1262IMLTRT, U3 BD2232G-GTR, U4 BD2232G-GTR, U5 RFswitch, U7 BD2232G-GTR, X1 12MHz, X2 FA-128_32.0000MF20X-K5, X3 32.768KHz

Commit message: OBC changed to STM32L4, pinout added, EPS ported
Parts:
- removed C42: 100nF, symbol COMMS-altium-import:3_100nF
- removed D1: VCC, symbol COMMS-altium-import:2_VCC
- removed U1: STM32L162RETx, Package_QFP:LQFP-64_10x10mm_P0.5mm, symbol MCU_ST_STM32L1:STM32L162RETx
- added C42: 100nF, symbol Device:C
- added D1: VCC, symbol Simulation_SPICE:DIODE
- added U1: STM32L476RGTx, Package_QFP:LQFP-64_10x10mm_P0.5mm, symbol MCU_ST_STM32L4:STM32L476RGTx
- C1, C10, C11, C12, C15, C16, C17, C18, C2, C27, C28, C31, C32, C33, C34, C35, C36, C37, C4, C40, C41, C5, C6, C7, C8, C9: CONTRIBUTOR danielCOMMS -> (none)
- C14: symbol COMMS-altium-import:3_1nF -> Device:C; CONTRIBUTOR danielCOMMS -> (none)
- C43, C44, C45: symbol COMMS-altium-import:0_1uF -> Device:C; CONTRIBUTOR danielCOMMS -> (none)
- R6: symbol COMMS-altium-import:3_10k -> Device:R
- R7, R8: symbol COMMS-altium-import:3_4.7k -> Device:R
Connections:
- net BUSY: now also U1.41 (PA8); no longer U2.14 (BUSY)
- net CHGOFF: now also U1.8 (PC0); no longer J2.7 (Pin_7)
- net CHRG: now also U1.28 (PB2)
- net CLPROG: now also U1.20 (PA4)
- net DIO1: now also U1.43 (PA10)
- net FAULT: now also U1.24 (PC4)
- net GND: now also C43.2, C44.2, C42.2, U1.12 (VSSA), U1.18 (VSS), U1.31 (VSS), U1.47 (VSS), U1.63 (VSS); no longer C43.1, C44.1
- net MISO: now also U1.35 (PB14)
- net MOSI: now also U1.36 (PB15)
- net MPPT_X: now also U1.22 (PA6)
- net MPPT_Y: now also U1.27 (PB1)
- net MPPT_Z: now also U1.23 (PA7)
- net NRST: now also C42.1, U1.7 (NRST)
- net OSC32_IN: now also U1.3 (PC14)
- net OSC32_OUT: now also U1.4 (PC15)
- net OSC_IN: now also U1.5 (PH0)
- net OSC_OUT: now also U1.6 (PH1)
- net P/L2BURN_OBC: no longer J3.1 (Pin_1)
- net P/L_POWER: no longer J4.5 (Pin_5)
- net PFO: now also U1.57 (PB5)
- net RST_DRIVERS: now also U1.42 (PA9)
- net SCK: now also U1.34 (PB13)
- net SCL: now also U1.58 (PB6)
- net SDA: now also U1.59 (PB7)
- net SEL_PH1: now also U1.44 (PA11)
- net SEL_PH2: now also U1.45 (PA12)
- net SEL_PH3: now also U1.10 (PC2); no longer J4.4 (Pin_4)
- net SWCLK: now also U1.49 (PA14)
- net SWDIO: now also U1.46 (PA13)
- net TOTAL_CURRENT: now also U1.14 (PA0)
- net VCC: now also C43.1, C44.1, J1.10 (Pin_10), D1.1 (A), U1.1 (VBAT), U1.13 (VDDA), U1.19 (VDD), U1.32 (VDD), U1.48 (VDDUSB), U1.64 (VDD); no longer C43.2, C44.2
- net VCC_TEST1: no longer J4.3 (Pin_3)
- net Boot0: now reaches R6.1
- net Boot0: now also U1.60 (BOOT0)
- net KILLSWITCH+: now reaches J1.4 (Pin_4)
- net BATT-: now reaches J1.6 (Pin_6)
- net ADC_PH1 renamed ADC_PH
- net ADC_PH: now also U1.25 (PC5)
- net ADC_PL2 renamed ADC_PL
- net ADC_PL: now also U1.15 (PA1)
- net BURNCOMMS_OBC renamed PoL_BURN_EN
- net PoL_BURN_EN: now also U1.30 (PB11)
- net DAC_PL2 renamed DAC_PL
- net DAC_PL: now also U1.21 (PA5)
- net HEATER renamed HEATER_PWR
- net NRESET renamed SX1262_NRST
- net SX1262_NRST: now also U1.40 (PC9)
- net NSS renamed SX1262_NSS
- net SX1262_NSS: now also U1.33 (PB12)
- net P/L_POWER_OBC renamed PoL_P/L_EN
- net PoL_P/L_EN: now also U1.11 (PC3)
- net PALE renamed STM32_PB3
- net STM32_PB3: now also U1.55 (PB3)
- net PCLK renamed STM32_PA2
- net STM32_PA2: now also U1.16 (PA2)
- net PDATA renamed STM32_PD2
- net STM32_PD2: now also U1.54 (PD2)
- net RST renamed EPS_RST
- net EPS_RST: now also U1.26 (PB0)
- net RX renamed UART_RX
- net UART_RX: now also U1.52 (PC11)
- net SEL renamed HEATER_EN
- net HEATER_EN: now also U1.29 (PB10)
- net TX renamed UART_TX
- net UART_TX: now also U1.51 (PC10)
- new net CHRGOFF: J2.7 (Pin_7)
- new net P/L_POWER: J4.5 (Pin_5)
- new net SEL_PH0: J4.4 (Pin_4)
- new net STM32_PA15: J3.1 (Pin_1), U1.50 (PA15)
- new net SX1262_BUSY: U2.14 (BUSY)
- new net VCC_UMBILICAL: D1.2 (K), J4.3 (Pin_3)
- no-connect marks 15 -> 14
Other:
- note added: "To be done in PL2 board"
- note added: "Umbilical Power Diode"
- note added: "Vcc Test"
- note added: "Vertical Connectors"
- note removed: "Clocks"
- moved on the sheet: C1, C10, C11, C12, C15, C16, C17, C18, C2, C27, C28, C31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

Commit message: hw revision, notes in MoM 09/11/2022
Other:
- note added: "PoL"
- note removed: "Current Limit Switch"
Changed lines of the file:
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@@
     (effects (font (size 1.524 1.524)) (justify left bottom))
   )
-  (text "Current Limit Switch" (at 326.39 142.24 0)
+  (text "PoL" (at 326.39 142.24 0)
     (effects (font (size 1.27 1.27)) (justify left bottom))
   )

Commit message: hw revision of OBC
Parts:
- removed C44: 1uF, symbol Device:C
- removed D1: VCC, symbol Simulation_SPICE:DIODE
- removed D2: VCC_TEST, symbol COMMS-altium-import:0_VCC_TEST
- removed J6: U.FL-R-SMT-1_10_, symbol COMMS-altium-import:1_U.FL-R-SMT-1_10_
- removed PROBE1: MS-156C, GGS_Connectors:CoaxialSwitch_Hirose_MS-156C3_Horizontal, symbol GGS_Connectors:MS-156C
- removed U4: BD2232G-GTR, symbol COMMS-altium-import:0_BD2232G-GTR
- added C?: 1uF, Capacitor_SMD:C_0603_1608Metric, symbol Device:C
- added D? (x2): D_Schottky, symbol Device:D_Schottky
- added J6: U.FL-R-SMT-1_10, Connector_Coaxial:U.FL_Hirose_U.FL-R-SMT-1_Vertical, symbol Connector:Conn_Coaxial
- added TP1: CoaxialSwitch_Testpoint, symbol Connector:CoaxialSwitch_Testpoint
- added U?: BD2232G-GTR, Package_SO:TSOP-5_1.65x3.05mm_P0.95mm, symbol COMMS-altium-import:0_BD2232G-GTR
- C1, C11, C12, C2, C4, C5, C6, C7, C8: footprint (none) -> Capacitor_SMD:C_0402_1005Metric
- C10, C9: footprint (none) -> Capacitor_SMD:C_0402_1005Metric; symbol COMMS-altium-import:3_3.3pF -> Device:C
- C14, C15, C16, C17, C18, C27, C28, C40, C41, C42, C43, C45: footprint (none) -> Capacitor_SMD:C_0603_1608Metric
- L1, L2, L3, L4, L5, L6: footprint (none) -> Inductor_SMD:L_0402_1005Metric
- L7: footprint (none) -> Inductor_SMD:L_0805_2012Metric
- R3, R4, R6, R7, R8: footprint (none) -> Resistor_SMD:R_0603_1608Metric
- U2: footprint (none) -> Package_DFN_QFN:QFN-24-1EP_4x4mm_P0.5mm_EP2.6x2.6mm
- U3, U7: footprint (none) -> Package_SO:TSOP-5_1.65x3.05mm_P0.95mm
Connections:
- net ADC_PH: now also J4.5 (Pin_5); no longer J4.6 (Pin_6)
- net ADC_PL: now also J2.9 (Pin_9); no longer J2.2 (Pin_2)
- net CHRG: now also J4.10 (Pin_10); no longer J4.1 (Pin_1)
- net CHRGOFF: now also J2.4 (Pin_4); no longer J2.7 (Pin_7)
- net CLPROG: now also J2.3 (Pin_3); no longer J2.8 (Pin_8)
- net DAC_PL: now also J2.8 (Pin_8); no longer J2.3 (Pin_3)
- net EPS_RST: no longer J3.10 (Pin_10)
- net FAULT: now also J4.9 (Pin_9); no longer J4.2 (Pin_2)
- net GND: now also C?.1, J6.2 (Ext), TP1.G, U?.2 (GND)
- net MPPT_X: no longer J2.9 (Pin_9)
- net MPPT_Y: no longer J4.8 (Pin_8)
- net MPPT_Z: no longer J4.9 (Pin_9)
- net NRST: now also J2.5 (Pin_5); no longer J2.6 (Pin_6)
- net P/L_POWER: now also J4.6 (Pin_6); no longer J4.5 (Pin_5)
- net RST_DRIVERS: now also J4.4 (Pin_4); no longer J4.7 (Pin_7)
- net SEL_PH0: now also J4.7 (Pin_7); no longer J4.4 (Pin_4)
- net SOLAR_X: now also J2.1 (Pin_1); no longer J2.10 (Pin_10)
- net SOLAR_Z: now also J4.1 (Pin_1); no longer J4.10 (Pin_10)
- net STM32_PA2: now also J2.10 (Pin_10); no longer J2.1 (Pin_1)
- net STM32_PD2: now also J4.2 (Pin_2); no longer J3.3 (Pin_3)
- net SWCLK: now also J2.7 (Pin_7); no longer J2.4 (Pin_4)
- net SWDIO: now also J2.6 (Pin_6); no longer J2.5 (Pin_5)
- net VCC: now also C?.2, D?.1 (K), D?.1 (K), U?.1 (IN); no longer J1.10 (Pin_10)
- net VCC_UMBILICAL: now also J4.8 (Pin_8), D?.2 (A); no longer J4.3 (Pin_3)
- net at L2.2: now also TP1.C
- net at C10.1, L5.2: now also J6.1 (In)
- net at C4.1, L1.2, L3.1: now also TP1.A
- new net 3V3_PERM: D?.2 (A), J1.10 (Pin_10)
- new net ADCS_POWER: U?.5 (OUT)
- new net BATT_NTC: J3.3 (Pin_3)
- new net PoL_ADCS_EN: U?.3 (EN/EN#)
Other:
- note added: "Low speed external Clock"
- note removed: "Low speed external"
- note removed: "To be done in PL2 board"
- note removed: "Vcc Test"
- moved on the sheet: C1, C11, C12, C14, C15, C16, C17, C18, C2, C27, C28, C38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
