File: pq_botboard/PQ_BotBoard/PQ_BotBoard.kicad_sch (KiCad schematic)
At the start: 28 parts, among them IC1 TCN75AVOA713, J1 53261-1471, J2 Conn_01x08_MountingPin, J3 53261-0271

Commit message: BOM creation schematic changes 2.0
Parts:
- D1: Manufacturer 1 (none) -> Advanced Photonix; Manufacturer Part Number 1 (none) -> SLCD-61N8; Supplier 1 (none) -> Farnell; Supplier Part Number 1 (none) -> 1218991
- H1, H2, H3, H4, H5, H6, NT1, NT2: Manufacturer 1 (none) -> N/A; Manufacturer Part Number 1 (none) -> N/A; Supplier 1 (none) -> N/A; Supplier Part Number 1 (none) -> N/A
- IC1: Manufacturer 1 (none) -> Microchip; Manufacturer Part Number 1 (none) -> TCN75AVOA; Supplier 1 (none) -> Mouser; Supplier Part Number 1 (none) -> 579-TCN75AVOA
- J1: Manufacturer Part Number 1 532611471 -> PicoBlade_53261-1571; Supplier 1 LCSC -> Mouser; Supplier Part Number 1 C505101 -> 538-53261-1571
- J2: Manufacturer 1 (none) -> MOLEX; Manufacturer Part Number 1 (none) -> PicoBlade_53398-0871; Supplier 1 (none) -> Mouser; Supplier Part Number 1 (none) -> 538-53398-0871
- J3: Manufacturer Part Number 1 532610271 -> _PicoBlade_53261-0271; Supplier 1 LCSC -> Mouser; Supplier Part Number 1 C189700 -> 538-53261-0271
- KS1: Supplier 1 LCSC -> Farnell; Supplier Part Number 1 C231335 -> 9901957
- KS2: Manufacturer Part Number 1 D2F-01L -> D2F-01L-A; Supplier 1 LCSC -> Farnell; Supplier Part Number 1 C231335 -> 1961083
- SC1: Manufacturer 1 (none) -> Azur Space; Manufacturer Part Number 1 (none) -> 3G30A; Supplier 1 (none) -> Lighttricity; Supplier Part Number 1 (none) -> N/A
Changed lines of the file:
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@@
+      (effects (font (size 1.27 1.27)) hide)
+    )
+    (property "Manufacturer 1" "N/A" (at 140.97 144.78 0)
+      (effects (font (size 1.27 1.27)) hide)
+    )
+    (property "Manufacturer Part Number 1" "N/A" (at 140.97 144.78 0)
+      (effects (font (size 1.27 1.27)) hide)
+    )
+    (property "Supplier 1" "N/A" (at 140.97 144.78 0)
+      (effects (font (size 1.27 1.27)) hide)
+    )
+    (property "Supplier Part Number 1" "N/A" (at 140.97 144.78 0)
       (effects (font (size 1.27 1.27)) hide)
     )
@@
       (effects (font (size 1.27 1.27)) hide)
     )
+    (property "Manufacturer 1" "N/A" (at 140.97 130.81 0)
+      (effects (font (size 1.27 1.27)) hide)
+    )
+    (property "Manufacturer Part Number 1" "N/A" (at 140.97 130.81 0)
+      (effects (font (size 1.27 1.27)) hide)
+    )
+    (property "Supplier 1" "N/A" (at 140.97 130.81 0)
+      (effects (font (size 1.27 1.27)) hide)
+    )
+    (property "Supplier Part Number 1" "N/A" (at 140.97 130.81 0)
+      (effects (font (size 1.27 1.27)) hide)
+    )
     (pin "1")
     (instances
@@
       (effects (font (size 1.27 1.27)) hide)
     )
-    (property "Manufacturer Part Number 1" "532610271" (at 107.95 104.14 0)
-      (effects (font (size 1.27 1.27)) hide)
-    )
-    (property "Supplier 1" "LCSC" (at 107.95 104.14 0)
-      (effects (font (size 1.27 1.27)) hide)
-    )
-    (property "Supplier Part Number 1" "C189700" (at 107.95 104.14 0)
+    (property "Manufacturer Part Number 1" "_PicoBlade_53261-0271" (at 107.95 104.14 0)
+      (effects (font (size 1.27 1.27)) hide)
+    )
+    (property "Supplier 1" "Mouser" (at 107.95 104.14 0)
+      (effects (font (size 1.27 1.27)) hide)
+    )
+    (property "Supplier Part Number 1" "538-53261-0271 " (at 107.95 104.14 0)
       (effects (font (size 1.27 1.27)) hide)
     )
@@
       (effects (font (size 1.27 1.27)) hide)
     )
+    (property "Manufacturer 1" "Advanced Photonix" (at 204.47 53.34 0)
+      (effects (font (size 1.27 1.27)) hide)
+    )
+    (property "Manufacturer Part Number 1" "SLCD-61N8" (at 204.47 53.34 0)
+      (effects (font (size 1.27 1.27)) hide)
+    )
+    (property "Supplier 1" "Farnell" (at 204.47 53.34 0)
+      (effects (font (size 1.27 1.27)) hide)
+    )
+    (property "Supplier Part Number 1" "1218991" (at 204.47 53.34 0)
+      (effects (font (size 1.27 1.27)) hide)
+    )
     (pin "1")
     (pin "2")
@@
       (effects (font (size 1.27 1.27)) hide)
     )
+    (property "Manufacturer 1" "N/A" (at 165.1 144.78 0)
+      (effects (font (size 1.27 1.27)) hide)
+    )
+    (property "Manufacturer Part Number 1" "N/A" (at 165.1 144.78 0)
+      (effects (font (size 1.27 1.27)) hide)
+    )
+    (property "Supplier 1" "N/A" (at 165.1 144.78 0)
+      (effects (font (size 1.27 1.27)) hide)
+    )
+    (property "Supplier Part Number 1" "N/A" (at 165.1 144.78 0)
+      (effects (font (size 1.27 1.27)) hide)
+    )
     (pin "1")
     (instances
@@
       (effects (font (size 1.27 1.27)) hide)
     )
+    (property "Manufacturer 1" "N/A" (at 189.23 144.78 0)
+      (effects (font (size 1.27 1.27)) hide)
+    )
+    (property "Manufacturer Part Number 1" "N/A" (at 189.23 144.78 0)
+      (effects (font (size 1.27 1.27)) hide)
+    )
+    (property "Supplier 1" "N/A" (at 189.23 144.78 0)
+      (effects (font (size 1.27 1.27)) hide)
+    )
+    (property "Supplier Part Number 1" "N/A" (at 189.23 144.78 0)
+      (effects (font (size 1.27 1.27)) hide)
+    )
     (pin "1")
     (instances
@@
     )
     (property "Datasheet" "~" (at 189.23 130.81 0)
+      (effects (font (size 1.27 1.27)) hide)
+    )
+    (property "Manufacturer 1" "N/A" (at 189.23 130.81 0)
+      (effects (font (size 1.27 1.27)) hide)
+    )
+    (property "Manufacturer Part Number 1" "N/A" (at 189.23 130.81 0)
+      (effects (font (size 1.27 1.27)) hide)
+    )
+    (property "Supplier 1" "N/A" (at 189.23 130.81 0)
+      (effects (font (size 1.27 1.27)) hide)
+    )
+    (property "Supplier Part Number 1" "N/A" (at 189.23 130.81 0)
       (effects (font (size 1.27 1.27)) hide)
     )
@@
       (effects (font (size 1.27 1.27)) hide)
     )
-    (property "Manufacturer Part Number 1" "D2F-01L" (at 107.95 140.97 0)
-      (effects (font (size 1.27 1.27)) hide)
-    )
-    (property "Supplier 1" "LCSC" (at 107.95 140.97 0)
-      (effects (font (size 1.27 1.27)) hide)
-    )
-    (property "Supplier Part Number 1" "C231335" (at 107.95 140.97 0)
+    (property "Manufacturer Part Number 1" "D2F-01L-A" (at 107.95 140.97 0)
+      (effects (font (size 1.27 1.27)) hide)
+    )
+    (property "Supplier 1" "Farnell" (at 107.95 140.97 0)
+      (effects (font (size 1.27 1.27)) hide)
+    )
+    (property "Supplier Part Number 1" "1961083" (at 107.95 140.97 0)
       (effects (font (size 1.27 1.27)) hide)
     )
@@
       (effects (font (size 1.27 1.27)) hide)
     )
+    (property "Manufacturer 1" "N/A" (at 152.4 48.26 0)
+      (effects (font (size 1.27 1.27)) hide)
+    )
+    (property "Manufacturer Part Number 1" "N/A" (at 152.4 48.26 0)
+      (effects (font (size 1.27 1.27)) hide)
+    )
+    (property "Supplier 1" "N/A" (at 152.4 48.26 0)
+      (effects (font (size 1.27 1.27)) hide)
+    )
+    (property "Supplier Part Number 1" "N/A" (at 152.4 48.26 0)
+      (effects (font (size 1.27 1.27)) hide)
+    )
     (pin "1")
     (pin "2")
@@
       (effects (font (size 1.27 1.27)) hide)
     )
-    (property "Manufacturer Part Number 1" "532611471" (at 82.55 88.9 0)
-      (effects (font (size 1.27 1.27)) hide)
-    )
-    (property "Supplier 1" "LCSC" (at 82.55 88.9 0)
-      (effects (font (size 1.27 1.27)) hide)
-    )
-    (property "Supplier Part Number 1" "C505101" (at 82.55 88.9 0)
+    (property "Manufacturer Part Number 1" "PicoBlade_53261-1571" (at 82.55 88.9 0)
+      (effects (font (size 1.27 1.27)) hide)
+    )
+    (property "Supplier 1" "Mouser" (at 82.55 88.9 0)
+      (effects (font (size 1.27 1.27)) hide)
+    )
+    (property "Supplier Part Number 1" "538-53261-1571 " (at 82.55 88.9 0)
       (effects (font (size 1.27 1.27)) hide)
     )
@@
       (effects (font (size 1.27 1.27)) hide)
     )
-    (property "Supplier 1" "LCSC" (at 91.44 140.97 0)
-      (effects (font (size 1.27 1.27)) hide)
-    )
-    (property "Supplier Part Number 1" "C231335" (at 91.44 140.97 0)
+    (property "Supplier 1" "Farnell" (at 91.44 140.97 0)
+      (effects (font (size 1.27 1.27)) hide)
+    )
+    (property "Supplier Part Number 1" "9901957 " (at 91.44 140.97 0)
       (effects (font (size 1.27 1.27)) hide)
     )
@@
     (property "BOM_MANUFACTURER PART" "" (at 152.4 87.63 0)
       (effects (font (size 1.27 1.27)) (justify left bottom) hide)
+    )
+    (property "Manufacturer 1" "Microchip" (at 152.4 87.63 0)
+      (effects (font (size 1.27 1.27)) hide)
+    )
+    (property "Manufacturer Part Number 1" "TCN75AVOA" (at 152.4 87.63 0)
+      (effects (font (size 1.27 1.27)) hide)
+    )
+    (property "Supplier 1" "Mouser" (at 152.4 87.63 0)
+      (effects (font (size 1.27 1.27)) hide)
+    )
+    (property "Supplier Part Number 1" " 579-TCN75AVOA" (at 152.4 87.63 0)
+      (effects (font (size 1.27 1.27)) hide)
     )
     (pin "1")
@@
       (effects (font (size 1.27 1.27)) hide)
     )
+    (property "Manufacturer 1" "Azur Space" (at 100.33 52.07 0)
+      (effects (font (size 1.27 1.27)) hide)
+    )
+    (property "Manufacturer Part Number 1" "3G30A" (at 100.33 52.07 0)
+      (effects (font (size 1.27 1.27)) hide)
+    )
+    (property "Supplier 1" "Lighttricity" (at 100.33 52.07 0)
+      (effects (font (size 1.27 1.27)) hide)
+    )
+    (property "Supplier Part Number 1" "N/A" (at 100.33 52.07 0)
+      (effects (font (size 1.27 1.27)) hide)
+    )
     (pin "1")
     (pin "2")
@@
     )
     (property "Datasheet" "~" (at 152.4 53.34 0)
+      (effects (font (size 1.27 1.27)) hide)
+    )
+    (property "Manufacturer 1" "N/A" (at 152.4 53.34 0)
+      (effects (font (size 1.27 1.27)) hide)
+    )
+    (property "Manufacturer Part Number 1" "N/A" (at 152.4 53.34 0)
+      (effects (font (size 1.27 1.27)) hide)
+    )
+    (property "Supplier 1" "N/A" (at 152.4 53.34 0)
+      (effects (font (size 1.27 1.27)) hide)
+    )
+    (property "Supplier Part Number 1" "N/A" (at 152.4 53.34 0)
       (effects (font (size 1.27 1.27)) hide)
     )
@@
     )
     (property "Datasheet" "~" (at 107.95 77.47 0)
+      (effects (font (size 1.27 1.27)) hide)
+    )
+    (property "Manufacturer 1" "MOLEX" (at 107.95 77.47 0)
+      (effects (font (size 1.27 1.27)) hide)
+    )
+    (property "Manufacturer Part Number 1" "PicoBlade_53398-0871" (at 107.95 77.47 0)
+      (effects (font (size 1.27 1.27)) hide)
+    )
+    (property "Supplier 1" "Mouser" (at 107.95 77.47 0)
+      (effects (font (size 1.27 1.27)) hide)
+    )
+    (property "Supplier Part Number 1" "538-53398-0871 " (at 107.95 77.47 0)
       (effects (font (size 1.27 1.27)) hide)
     )
@@
       (effects (font (size 1.27 1.27)) hide)
     )
+    (property "Manufacturer 1" "N/A" (at 165.1 130.81 0)
+      (effects (font (size 1.27 1.27)) hide)
+    )
+    (property "Manufacturer Part Number 1" "N/A" (at 165.1 130.81 0)
+      (effects (font (size 1.27 1.27)) hide)
+    )
+    (property "Supplier 1" "N/A" (at 165.1 130.81 0)
+      (effects (font (size 1.27 1.27)) hide)
+    )
+    (property "Supplier Part Number 1" "N/A" (at 165.1 130.81 0)
+      (effects (font (size 1.27 1.27)) hide)
+    )
