File: pq_botboard/PQ_BotBoard/PQ_BotBoard.kicad_sch (KiCad schematic)
At the start: 37 parts, among them IC1 TCN75AVOA713, J1 53261-1471, J2 Conn_01x08_MountingPin, J5 Conn_01x03_MountingPin, U1 TPS7A7002DDAR

Commit message: add Lighticity SC to bottom with the option to solder using epoxy
Parts:
- removed SC1: ~, power-nsl:Lighttricity_S3040_CIC, symbol power-nsl:S3040_CIC
- added SC2: ~, power-nsl:Lighttricity_S3040_CIC, symbol power-nsl:S3040_CIC
Connections:
- net GND: now also SC2.1
- net SOLAR_Y: now also SC2.3
Other:
- moved on the sheet: D2
Changed lines of the file:
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@@
   (no_connect (at 110.49 146.05))
   (no_connect (at 92.71 146.05))
+  (wire (pts (xy 162.56 50.8) (xy 170.18 50.8))
+    (stroke (width 0) (type default))
+  )
   (wire (pts (xy 114.3 87.63) (xy 113.03 87.63))
     (stroke (width 0) (type default))
@@
     (stroke (width 0.254) (type default))
   )
+  (wire (pts (xy 107.95 49.53) (xy 115.57 49.53))
+    (stroke (width 0) (type default))
+  )
   (wire (pts (xy 232.41 55.88) (xy 234.95 55.88))
     (stroke (width 0) (type default))
@@
     (stroke (width 0) (type default))
   )
-  (wire (pts (xy 144.78 50.8) (xy 151.13 50.8))
-    (stroke (width 0) (type default))
-  )
   (wire (pts (xy 182.88 107.95) (xy 191.77 107.95))
     (stroke (width 0) (type default))
@@
   )
   (polyline (pts (xy 236.22 80.01) (xy 273.05 80.01))
+    (stroke (width 0) (type default))
+  )
+  (wire (pts (xy 95.25 49.53) (xy 87.63 49.53))
     (stroke (width 0) (type default))
   )
@@
     (stroke (width 0) (type default))
   )
+  (wire (pts (xy 144.78 50.8) (xy 154.94 50.8))
+    (stroke (width 0) (type default))
+  )
   (wire (pts (xy 148.59 92.71) (xy 152.4 92.71))
     (stroke (width 0.254) (type default))
@@
     (stroke (width 0) (type default))
   )
-  (wire (pts (xy 87.63 50.8) (xy 96.52 50.8))
-    (stroke (width 0) (type default))
-  )
   (polyline (pts (xy 76.2 58.42) (xy 129.54 58.42))
     (stroke (width 0) (type default))
   )
-  (wire (pts (xy 104.14 50.8) (xy 114.554 50.8))
+  (wire (pts (xy 87.63 49.53) (xy 87.63 50.8))
     (stroke (width 0) (type default))
   )
@@
   )
   (wire (pts (xy 172.72 72.39) (xy 144.78 72.39))
-    (stroke (width 0) (type default))
-  )
-  (wire (pts (xy 158.75 50.8) (xy 170.18 50.8))
     (stroke (width 0) (type default))
   )
@@
     (effects (font (size 1.27 1.27)) (justify right bottom))
   )
-  (label "SOLAR_Y" (at 114.554 50.8 0) (fields_autoplaced)
+  (label "SOLAR_Y" (at 115.57 49.53 0) (fields_autoplaced)
     (effects (font (size 1.27 1.27)) (justify left bottom))
   )
@@
     )
   )
-  (symbol (lib_id "Device:LED") (at 154.94 50.8 180) (unit 1)
+  (symbol (lib_id "Device:LED") (at 158.75 50.8 180) (unit 1)
     (in_bom yes) (on_board yes) (dnp no)
-    (property "Reference" "D2" (at 151.13 45.72 0)
-      (effects (font (size 1.27 1.27)))
-    )
-    (property "Value" "LED" (at 151.13 48.26 0)
-      (effects (font (size 1.27 1.27)))
-    )
-    (property "Footprint" "LED_SMD:LED_0402_1005Metric" (at 154.94 50.8 0)
-      (effects (font (size 1.27 1.27)) hide)
-    )
-    (property "Datasheet" "~" (at 154.94 50.8 0)
+    (property "Reference" "D2" (at 154.94 45.72 0)
+      (effects (font (size 1.27 1.27)))
+    )
+    (property "Value" "LED" (at 154.94 48.26 0)
+      (effects (font (size 1.27 1.27)))
+    )
+    (property "Footprint" "LED_SMD:LED_0402_1005Metric" (at 158.75 50.8 0)
+      (effects (font (size 1.27 1.27)) hide)
+    )
+    (property "Datasheet" "~" (at 158.75 50.8 0)
       (effects (font (size 1.27 1.27)) hide)
     )
@@
     )
   )
-  (symbol (lib_id "power-nsl:S3040_CIC") (at 100.33 50.8 270) (unit 1)
-    (in_bom yes) (on_board yes) (dnp no) (fields_autoplaced)
-    (property "Reference" "SC1" (at 100.965 45.72 90)
-      (effects (font (size 1.27 1.27)))
-    )
-    (property "Value" "~" (at 100.33 50.8 0)
-      (effects (font (size 1.27 1.27)))
-    )
-    (property "Footprint" "power-nsl:Lighttricity_S3040_CIC" (at 100.33 50.8 0)
-      (effects (font (size 1.27 1.27)) hide)
-    )
-    (property "Datasheet" "" (at 100.33 50.8 0)
-      (effects (font (size 1.27 1.27)) hide)
-    )
-    (pin "1")
-    (pin "2")
-    (instances
-      (project "PQ_BotBoard"
-        (path "/e40a5bef-c31a-474e-b379-53d1d13d8a60"
-          (reference "SC1") (unit 1)
-        )
-      )
-    )
-  )
   (symbol (lib_id "symbols-nsl:Silkscreen_Annotation") (at 242.57 115.57 0) (unit 1)
     (in_bom yes) (on_board yes) (dnp no) (fields_autoplaced)
@@
         )
       )
+    )
+  )
+  (symbol (lib_name "S3040_CIC_1") (lib_id "power-nsl:S3040_CIC") (at 101.6 49.53 270) (unit 1)
+    (in_bom yes) (on_board yes) (dnp no) (fields_autoplaced)
+    (property "Reference" "SC2" (at 101.6 41.91 90)
+      (effects (font (size 1.27 1.27)))
+    )
+    (property "Value" "~" (at 101.6 49.53 0)
+      (effects (font (size 1.27 1.27)))
+    )
+    (property "Footprint" "power-nsl:Lighttricity_S3040_CIC" (at 101.6 49.53 0)
+      (effects (font (size 1.27 1.27)) hide)
+    )
+    (property "Datasheet" "" (at 101.6 49.53 0)
+      (effects (font (size 1.27 1.27)) hide)
+    )
+    (pin "3")
+    (pin "1")
+    (pin "2")
+    (instances
+      (project "PQ_BotBoard"
+        (path "/e40a5bef-c31a-474e-b379-53d1d13d8a60"
+          (reference "SC2") (unit 1)
+        )
+      )

Commit message: Botboards and Latbaords corrected and revised. Production ready
Parts:
- removed H3, H4: MountingHole_Pad, MountingHole:MountingHole_2.2mm_M2_Pad, symbol Mechanical:MountingHole_Pad
- removed J5: Conn_01x03_MountingPin, Connector_Molex:Molex_PicoBlade_53261-0371_1x03-1MP_P1.25mm_Horizontal, symbol Connector_Generic_MountingPin:Conn_01x03_MountingPin
- D3, SC2: value ~ -> (none)
- U1: value TPS7A7002DDAR -> TPS7A7002DDAR
Connections:
- no-connect marks 2 -> 3
