File: pq_botboard/PQ_BotBoard/PQ_BotBoard.kicad_pcb (KiCad board)
At the start: 6 copper layers, 64 x 52 mm, 37 parts, among them IC1 TCN75AVOA713, J1 53261-1471, J2 Conn_01x08_MountingPin, J5 Conn_01x03_MountingPin, U1 TPS7A7002DDAR

Commit message: add missing component names and relocate others
Other:
- board text added: "J5"
Changed lines of the file:
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@@
     (property "ki_keywords" "connector")
     (attr smd)
-    (fp_text reference "J5" (at 0 -4.4 90) (layer "F.SilkS")
+    (fp_text reference "J5" (at 0 -4.4 90) (layer "F.SilkS") hide
         (effects (font (size 1 1) (thickness 0.15)))
     )
@@
     (property "ki_keywords" "cap capacitor")
     (attr smd)
-    (fp_text reference "C2" (at 2.032 0 unlocked) (layer "F.SilkS")
+    (fp_text reference "C2" (at -1.9245 -0.0124 unlocked) (layer "F.SilkS")
         (effects (font (size 0.4 0.4) (thickness 0.15)))
     )
@@
     (effects (font (size 2 2) (thickness 0.3) bold) (justify bottom mirror))
   )
+  (gr_text "J5" (at 97.2312 47.117) (layer "F.SilkS")
+    (effects (font (size 0.4 0.4) (thickness 0.1)))
+  )
   (gr_text "+Z" (at 61.9008 57.6088) (layer "Cmts.User")
