File: pq_latboard/PQ_Lat_Board/PQ_Lat_Board.kicad_sch (KiCad schematic)
At the start: 27 parts, among them IC1 TCN75AVOA713, J1 Conn_01x11_MountingPin, J2 Conn_Coaxial

Commit message: Recenter holes in Lateral PCB as there was a slight misalignment with the top structure
Parts:
- TK1: renamed from THT1; value 7.5 -> 4.7
Changed lines of the file:
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@@
   (symbol (lib_id "Device:R") (at 81.28 64.77 90) (unit 1)
     (in_bom yes) (on_board yes) (dnp no) (fields_autoplaced)
-    (property "Reference" "THT1" (at 81.28 59.69 90)
+    (property "Reference" "TK1" (at 81.28 59.69 90)
       (effects (font (size 1.27 1.27)))
     )
-    (property "Value" "7.5" (at 81.28 62.23 90)
+    (property "Value" "4.7" (at 81.28 62.23 90)
       (effects (font (size 1.27 1.27)))
     )
@@
       (project "PQ_Lat_Board"
         (path "/4da848d5-e65a-4ace-88f8-d9d6d6b9afa2"
-          (reference "THT1") (unit 1)
+          (reference "TK1") (unit 1)
         )
       )

Commit message: lateral modification
Parts:
- removed D2: LED, LED_SMD:LED_0402_1005Metric, symbol Device:LED
Connections:
- net PH- is gone; now on net GND: D1.1, J1.7 (Pin_7)
- net VCC_MAG is gone; now on net ADCS: J1.3 (Pin_3)
