File: pq_botboard/PQ_BotBoard - copia/PQ_BotBoard.kicad_sch (KiCad schematic)
At the start: 37 parts, among them IC1 TCN75AVOA713, J1 53261-1471, J2 Conn_01x08_MountingPin, J5 Conn_01x03_MountingPin, U1 TPS7A7002DDAR

Commit message: Removed photodiode +Y magnetorquer PCB
Parts:
- NT1: footprint (none) -> NetTie:NetTie-2_SMD_Pad0.5mm
Changed lines of the file:
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@@
 			)
 		)
-		(property "Footprint" ""
+		(property "Footprint" "NetTie:NetTie-2_SMD_Pad0.5mm"
 			(at 157.48 50.8 0)
 			(effects
