File: pq_adcs/PQ_ADCS_HBridge/PQ_ADCS.kicad_sch (KiCad schematic)
At the start: 53 parts, among them J1 CES-110-02-L-S, J10 Conn_01x03_MountingPin, J11 Conn_01x09_MountingPin, J12 CES-102-02-L-S, J13 Conn_01x15_MountingPin, J2 CES-110-02-L-S, J3 CES-110-02-L-S, J4 CES-110-02-L-S, J6 Conn_01x10_MountingPin, J7 Conn_01x10_MountingPin, J8 Conn_01x10_MountingPin, J9 Conn_01x10_MountingPin, U1 LPV542, U2 LPV542, U3 LPV542, U4 IIM-42652, U5 DRV8214RTER, U6 TMUX1108RSVR, U7 MMC5983MA, U8 DRV8214RTER, U9 DRV8214RTER

Commit message: Hbridge
Parts:
- removed J10: Conn_01x03_MountingPin, Connector_Molex:Molex_PicoBlade_53261-0371_1x03-1MP_P1.25mm_Horizontal, symbol Connector_Generic_MountingPin:Conn_01x03_MountingPin
- removed J11: Conn_01x09_MountingPin, Connector_Molex:Molex_PicoBlade_53261-0971_1x09-1MP_P1.25mm_Horizontal, symbol Connector_Generic_MountingPin:Conn_01x09_MountingPin
- removed J13: Conn_01x15_MountingPin, Connector_Molex:Molex_PicoBlade_53261-1571_1x15-1MP_P1.25mm_Horizontal, symbol Connector_Generic_MountingPin:Conn_01x15_MountingPin
- removed J6, J7, J8, J9: Conn_01x10_MountingPin, Connector_Molex:Molex_PicoBlade_53261-1071_1x10-1MP_P1.25mm_Horizontal, symbol Connector_Generic_MountingPin:Conn_01x10_MountingPin
- added J5, J6, J7, J8: 53261-1471, Connector_Molex:Molex_PicoBlade_53261-1571_1x15-1MP_P1.25mm_Horizontal, symbol Connector_Generic_MountingPin:Conn_01x15_MountingPin
Connections:
- net +MAG+X: now also J6.8 (Pin_8)
- net +MAG+Z: now also J7.8 (Pin_8)
- net +MAG-X: now also J5.10 (Pin_10), J6.9 (Pin_9)
- net +MAG-Y: now also J8.2 (Pin_2)
- net +MAG-Z: now also J5.1 (Pin_1), J7.9 (Pin_9)
- net -MAG-X: now also J5.11 (Pin_11)
- net -MAG-Y: now also J8.3 (Pin_3)
- net -MAG-Z: now also J5.2 (Pin_2)
- net 3V3_PERM: now also J5.12 (Pin_12), J5.3 (Pin_3), J6.10 (Pin_10), J7.10 (Pin_10), J7.3 (Pin_3), J8.4 (Pin_4)
- net BATT-: now also J8.10 (Pin_10)
- net BATT_NTC: now also J6.5 (Pin_5)
- net BURNCOMMS: now also J6.3 (Pin_3), J6.4 (Pin_4)
- net GND: now also J5.15 (Pin_15), J5.6 (Pin_6), J5.8 (Pin_8), J5.MP (MountPin), J6.13 (Pin_13), J6.15 (Pin_15), J6.MP (MountPin), J7.13 (Pin_13), J7.15 (Pin_15), J7.2 (Pin_2), J7.6 (Pin_6), J7.MP (MountPin), J8.7 (Pin_7), J8.MP (MountPin)
- net HEATER_PWR: now also J6.6 (Pin_6)
- net KILLSWITCH+: now also J8.11 (Pin_11)
- net NRST: now also J8.12 (Pin_12)
- net PHT2: now also J6.14 (Pin_14)
- net PHT3: now also J5.7 (Pin_7)
- net PHT4: now also J7.14 (Pin_14)
- net PHT5: now also J8.8 (Pin_8)
- net SCL3: now also J5.14 (Pin_14), J5.5 (Pin_5), J6.12 (Pin_12), J7.12 (Pin_12), J7.5 (Pin_5), J8.6 (Pin_6)
- net SDA3: now also J5.13 (Pin_13), J5.4 (Pin_4), J6.11 (Pin_11), J7.11 (Pin_11), J7.4 (Pin_4), J8.5 (Pin_5)
- net SOLAR_X: now also J5.9 (Pin_9), J6.7 (Pin_7)
- net SOLAR_Y: now also J7.1 (Pin_1), J8.1 (Pin_1)
- net SOLAR_Z: now also J6.1 (Pin_1), J7.7 (Pin_7)
- net SWCLK: now also J8.13 (Pin_13)
- net SWDIO: now also J8.14 (Pin_14)
- net SWO: now also J8.9 (Pin_9)
- net VCC_UMBILICAL: now also J8.15 (Pin_15)
Other:
- note added: "+X all pins included"
- note added: "+Z all pins included (excluded burncomms) +Y Included all pins (excluded burncomms)"
- note added: "-Y Included all pins"
- note added: "PAYLOAD Burncomms"
- moved on the sheet: Annotation1, Annotation2, C10, C15, C2, C3, C4, C5, C6, C7, C8, C9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

Commit message: Trying to add connectors bottom ADCS PCB
Connections:
- net +MAG+X: now also J5.9 (Pin_9); no longer J6.8 (Pin_8)
- net +MAG+Z: now also J7.2 (Pin_2); no longer J7.8 (Pin_8)
- net +MAG-X: now also J7.9 (Pin_9); no longer J6.9 (Pin_9)
- net +MAG-Z: now also J5.2 (Pin_2), J7.3 (Pin_3); no longer J5.1 (Pin_1), J7.9 (Pin_9)
- net -MAG-X: now also J7.10 (Pin_10); no longer J5.11 (Pin_11)
- net -MAG-Z: now also J5.3 (Pin_3); no longer J5.2 (Pin_2)
- net 3V3_PERM: now also J5.11 (Pin_11), J5.4 (Pin_4), J6.8 (Pin_8), J7.11 (Pin_11), J7.4 (Pin_4); no longer J5.12 (Pin_12), J5.3 (Pin_3), J6.10 (Pin_10), J7.10 (Pin_10), J7.3 (Pin_3)
- net BATT_NTC: now also J6.12 (Pin_12)
- net GND: now also J6.11 (Pin_11), J7.8 (Pin_8); no longer J5.6 (Pin_6), J6.15 (Pin_15), J7.13 (Pin_13), J7.2 (Pin_2), J7.6 (Pin_6)
- net PHT1: now also J7.14 (Pin_14)
- net PHT2: now also J5.14 (Pin_14); no longer J6.14 (Pin_14)
- net PHT4: now also J7.7 (Pin_7); no longer J7.14 (Pin_14)
- net SCL3: now also J5.13 (Pin_13), J5.6 (Pin_6), J6.10 (Pin_10), J7.13 (Pin_13), J7.6 (Pin_6); no longer J5.14 (Pin_14), J5.5 (Pin_5), J6.12 (Pin_12), J7.12 (Pin_12), J7.5 (Pin_5)
- net SDA3: now also J5.12 (Pin_12), J5.5 (Pin_5), J6.9 (Pin_9), J7.12 (Pin_12), J7.5 (Pin_5); no longer J5.13 (Pin_13), J5.4 (Pin_4), J6.11 (Pin_11), J7.11 (Pin_11), J7.4 (Pin_4)
- net SOLAR_X: now also J6.1 (Pin_1), J6.15 (Pin_15); no longer J5.9 (Pin_9), J6.7 (Pin_7)
- net SOLAR_Y: now also J6.7 (Pin_7); no longer J7.1 (Pin_1)
- net SOLAR_Z: now also J5.1 (Pin_1), J7.1 (Pin_1); no longer J6.1 (Pin_1), J7.7 (Pin_7)
- new net HEATER_NTC: J6.14 (Pin_14)
