File: pq_botboard - editado/PQ_BotBoard/PQ_BotBoard.kicad_pcb (KiCad board)
At the start: 6 copper layers, 64 x 52 mm, 38 parts, among them IC1 TCN75AVOA713, J1 53261-1471, J2 Conn_01x08_MountingPin, U1 TPS7A7002DDAR

Commit message: Botboard corrected. Need to be verified
Parts:
- moved C2 1.49 mm to (99.0, 49.0), turned to 90 degrees
Routing:
- net /VCC_MAG: track 9829.9 -> 9782.2 mm
- net GND: track 15.9 -> 34.1 mm, vias 20 -> 28
- net /PH+: track 98.8 -> 82.1 mm
- net /BATT-: track 148.6 -> 146.3 mm
- net /SWCLK: track 39.3 -> 38.0 mm
- net /BATT+: track 60.9 -> 59.6 mm
- net /VCC: track 52.4 -> 51.4 mm
- net Net-(U1-EN): track 24.9 -> 24.3 mm
- net /SOLAR_Y: vias 4 -> 1
