File: pq_botnotsobot/PQ_Botnotsobot/PQ_Botnotsobot.kicad_sch (KiCad schematic)
At the start: 18 parts, among them J1 D2FLA, J2 D2FLA1

Commit message: Botboards and Latbaords corrected and revised. Production ready
Parts:
- removed H3, H4: MountingHole_Pad, MountingHole:MountingHole_2.2mm_M2_Pad, symbol Mechanical:MountingHole_Pad
Connections:
- no-connect marks 12 -> 10
