File: pq_latboard_deploy/PQ_Lat_Board_Deploy.kicad_pcb (KiCad board)
At the start: 6 copper layers, 48 x 48 mm, 26 parts, among them IC1 TCN75AVOA713, J1 Conn_01x11_MountingPin, J2 Conn_Coaxial

Commit message: Botboards and Latbaords corrected and revised. Production ready
Parts:
- removed H5: MountingHole_Pad, MountingHole:MountingHole_2.2mm_M2_DIN965_Pad_TopOnly
- removed J2: Conn_Coaxial, Connector_Coaxial:U.FL_Hirose_U.FL-R-SMT-1_Vertical
- added R1: WHA5R0FET, WHA5R0FET:RESAD1524W60L508D254, F.Cu at (79.1, 71.7)
- added R2: WHA5R0FET, WHA5R0FET:RESAD1524W60L508D254, F.Cu at (79.5, 75.1)
- moved C1 3.17 mm to (101.2, 47.6), turned to 180 degrees
- moved H4 0.40 mm to (79.0, 84.4)
Routing:
- net /BURNCOMMS: track 0.00 -> 55.9 mm
- net /Antenna Connector: track 4.41 -> 0.00 mm
- net /VCC: track 31.7 -> 34.1 mm, vias 0 -> 2
- removed copper zone on F.Cu, net /Antenna Connector
Other:
- outline, holes or cut-outs redrawn
