File: pq_latboard_deploy/PQ_Lat_Board_Deploy.kicad_sch (KiCad schematic)
At the start: 26 parts, among them IC1 TCN75AVOA713, J1 Conn_01x11_MountingPin, J2 Conn_Coaxial

Commit message: Botboards and Latbaords corrected and revised. Production ready
Parts:
- removed H5: MountingHole_Pad, MountingHole:MountingHole_2.2mm_M2_DIN965_Pad_TopOnly, symbol Mechanical:MountingHole_Pad
- removed J2: Conn_Coaxial, Connector_Coaxial:U.FL_Hirose_U.FL-R-SMT-1_Vertical, symbol Connector:Conn_Coaxial
- added R1, R2: WHA5R0FET, WHA5R0FET:RESAD1524W60L508D254, symbol WHA5R0FET:WHA5R0FET
Connections:
- net BURNCOMMS: now also R1.1, R2.1
- net GND: now also R1.2, R2.2
Other:
- note added: "COMMS antenna thermal knife"
- note removed: "COMMS antenna coaxial connector"
- moved on the sheet: Annotation1, Annotation2, Annotation3, Annotation4, Annotation5, Annotation6, Annotation7, Annotation8, H1, H2, H3, H4
