File: pq_obc_comms/pq_obc_comms/pq_obc_comms.kicad_sch (KiCad schematic)
At the start: 69 parts, among them J1 Conn_01x10, J2 Conn_01x10, J3 Conn_01x10, J4 Conn_01x10, J6 U.FL, U1 STM32L476RGTx, U2 SX1262IMLTRT, U3 BD2232G-GTR, U4 BD2232G-GTR, U5 BGS12PL6E6327XTSA1, U6 BD2232G-GTR, U7 BD2232G-GTR, X1 ECS-120-18-33-JEM-TR3, X2 FA-128_32.0000MF20X-K5, X3 ABS09-32.768KHZ-7-T

Commit message: obccomms_pol_pulldows added. production ready
Parts:
- added R10, R11, R12, R9: 10k, Resistor_SMD:R_0402_1005Metric, symbol Device:R
Connections:
- net GND: now also R10.2, R11.1, R12.1, R9.1
- net HEATER_EN: now also R12.2
- net PoL_ADCS_POWER_EN: now also R10.1
- net PoL_BURN_EN: now also R11.2
- net PoL_P/L_EN: now also R9.2
